File: cad_files/drv8825_stepper.kicad_pcb (KiCad board)
At the start: 2 copper layers, 49 x 65 mm, 59 parts, among them J1 USB_C_Receptacle_USB2.0, J10 Conn_01x03, J11 Conn_01x03, J12 Conn_01x02, J2 RJ11, J3 RJ11, J4 PH, J5 PH, J6 Conn_02x03_Odd_Even, J7 Conn_01x04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

Commit message: update cad
Parts:
- removed J8: Conn_01x12, Connector_Molex:Molex_Mini-Fit_Jr_5569-12A2_2x06_P4.20mm_Horizontal
- added D8: LED, LED_SMD:LED_0603_1608Metric, F.Cu at (125.2, 112.0)
- added D9: LED, LED_SMD:LED_0603_1608Metric, F.Cu at (125.2, 115.0)
- added R12: 15k, Resistor_SMD:R_0603_1608Metric, F.Cu at (121.9, 110.2)
- added R13: 15k, Resistor_SMD:R_0603_1608Metric, F.Cu at (118.0, 112.5)
- added SW2: SW_Push, EvezorLIB:SWITCH_2x3_SMD_TACTILE_GREEN, F.Cu at (114.5, 116.3)
- added SW3: SW_Push, EvezorLIB:SWITCH_2x3_SMD_TACTILE_GREEN, F.Cu at (121.0, 116.3)
- J10, J11: footprint Connector_JST:JST_XH_B3B-XH-AM_1x03_P2.50mm_Vertical -> Connector_JST:JST_XH_S3B-XH-A-1_1x03_P2.50mm_Horizontal
- J7: footprint Connector_Molex:Molex_KK-254_AE-6410-04A_1x04_P2.54mm_Vertical -> Connector_JST:JST_XH_S4B-XH-A_1x04_P2.50mm_Horizontal
- J9: footprint Connector_JST:JST_PH_B5B-PH-SM4-TB_1x05-1MP_P2.00mm_Vertical -> Connector_JST:JST_PH_B5B-PH-K_1x05_P2.00mm_Vertical
- R8, R9: value 0.33 -> 0.1; footprint Resistor_SMD:R_0603_1608Metric -> Resistor_SMD:R_0805_2012Metric
- TP1: value MOTOR_CURRENT -> MCTP
- moved J10 75.0 mm to (109.5, 79.0), turned to 180 degrees
- moved J11 61.6 mm to (121.0, 79.0), turned to 180 degrees
- moved J9 59.9 mm to (136.5, 87.4), turned to 180 degrees
- moved J7 49.5 mm to (135.0, 80.5), turned to 180 degrees
- moved C7 48.5 mm to (138.1, 95.0)
- moved C12 44.5 mm to (138.1, 92.5), turned to 180 degrees
- moved R10 43.1 mm to (133.8, 114.6), turned to 180 degrees
- moved R9 41.9 mm to (122.5, 88.4)
- moved R11 41.5 mm to (133.8, 112.5), turned to 180 degrees
- moved R8 36.0 mm to (119.5, 88.4), turned to 90 degrees
- moved REF** 35.1 mm to (139.0, 118.2)
- moved R6 33.7 mm to (118.4, 107.0)
- moved C11 32.6 mm to (129.5, 93.7), turned to 270 degrees
- moved R7 31.7 mm to (118.4, 108.8)
- moved C15 28.6 mm to (126.5, 91.5)
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Connections:
- C14 pad 1: Net-(C14-Pad1) -> /V3P3
- J10 pad 1: /MAX -> /MIN
- J11 pad 1: /MIN -> /MAX
- R6 pad 1: Net-(R6-Pad1) -> /V3P3
- R7 pad 1: Net-(R7-Pad1) -> /V3P3
- RV1 pad 2: Net-(RV1-Pad2) -> /CURRENT_REF
- TP1 pad 1: Net-(RV1-Pad2) -> /CURRENT_REF
- U3 pad 10: /M0 -> /FAULT
- U3 pad 11: /ENABLE -> /SLEEP
- U3 pad 14: /MAX -> /ENCDR_NEO
- U3 pad 15: /MIN -> Net-(U3-Pad15)
- U3 pad 3: /STEP -> /M2
- U3 pad 30: Net-(U3-Pad30) -> /LED_2
- U3 pad 31: Net-(U3-Pad31) -> /LED_1
- U3 pad 32: Net-(U3-Pad32) -> /BUTTON_2
- U3 pad 33: Net-(U3-Pad33) -> /BUTTON_1
- U3 pad 37: Net-(U3-Pad37) -> /HOME
- U3 pad 39: Net-(U3-Pad39) -> /S_RESET
- U3 pad 4: /DIR -> /M1
- U3 pad 40: Net-(U3-Pad40) -> /MIN
- U3 pad 41: Net-(U3-Pad41) -> /MAX
- U3 pad 42: Net-(U3-Pad42) -> /CURRENT_REF
- U3 pad 5: /DECAY -> /M0
- U3 pad 6: /SLEEP -> /STEP
- U3 pad 7: /S_RESET -> /ENABLE
- U3 pad 8: /M2 -> /DIR
- U3 pad 9: /M1 -> /DECAY
- U4 pad 10: Net-(J7-Pad2) -> Net-(J7-Pad4)
- U4 pad 12: Net-(RV1-Pad2) -> /CURRENT_REF
- U4 pad 13: Net-(RV1-Pad2) -> /CURRENT_REF
- U4 pad 15: Net-(C14-Pad1) -> /V3P3
- U4 pad 18: Net-(R6-Pad1) -> /FAULT
- U4 pad 27: Net-(R7-Pad1) -> /HOME
- U4 pad 5: Net-(J7-Pad3) -> Net-(J7-Pad1)
- U4 pad 7: Net-(J7-Pad4) -> Net-(J7-Pad2)
- U4 pad 8: Net-(J7-Pad1) -> Net-(J7-Pad3)
Routing:
- net +3V3: track 82.8 -> 164.6 mm, vias 2 -> 6
- net /SDA: track 0.00 -> 47.2 mm, vias 0 -> 2
- net /V_MOTOR: track 0.00 -> 44.5 mm, vias 0 -> 9
- net /SCL: track 0.00 -> 41.2 mm, vias 0 -> 2
- net /ENCDR_NEO: track 0.00 -> 37.4 mm, vias 0 -> 2
- net /MAX: track 0.00 -> 30.3 mm, vias 0 -> 1
- net /MIN: track 0.00 -> 27.9 mm, vias 0 -> 1
- net /FAULT: track 0.00 -> 26.6 mm, vias 0 -> 3
- net Net-(J7-Pad2): track 0.00 -> 24.3 mm
- net /SLEEP: track 0.00 -> 24.0 mm, vias 0 -> 1
- net /CURRENT_REF: track 0.00 -> 23.8 mm, vias 0 -> 1
- net Net-(J7-Pad1): track 0.00 -> 23.5 mm
- net Net-(J7-Pad4): track 0.00 -> 23.4 mm
- net /HOME: track 0.00 -> 23.3 mm, vias 0 -> 3
- net Net-(J7-Pad3): track 0.00 -> 22.1 mm
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- added copper zone on B.Cu, net /V_MOTOR
- added copper zone on F.Cu, net /V_MOTOR
Other:
- board size 49 x 65 mm -> 49 x 80 mm
- board text added: "1"
- board text added: "2"
- board text added: "DRV8825 STEPPER DRIVER V1.0"
- board text added: "ENCODER"
- board text added: "MAX"
- board text added: "MIN"
- board text added: "POWER INPUT"
- board text added: "STEPPER"
- board text removed: "THE THING V1.0P"
- board text removed: "www.evezor.com/products/thisProduct"
